Commit message: Update cube.urdf

File: cube.urdf (robot description, URDF)
Before this commit: robot simple_cube, 1 links, 0 joints
Links:
- removed link base_link
- added link cube; visual box size=1 1 1
Joints:
- added joint fixed_joint: type fixed, parent base_link, child cube, origin xyz=0 0 0.5
